File: mcu_pfc.kicad_sch (KiCad schematic)
At the start: 11 parts, among them Q5 FGA60N65SMD, U6 STM32F103C8Tx, Y1 8MHz

Commit message: added progress
Parts:
- removed R3: R, symbol Device:R
- added R3: 4m, symbol Device:R_Shunt
- C1, C2: footprint (none) -> Capacitor_SMD:C_0805_2012Metric
- C3: value C_Polarized_US -> 330u; footprint (none) -> Capacitor_THT:CP_Radial_D35.0mm_P10.00mm_3pin_SnapIn
- L1: value L -> 470uH
- R2: footprint (none) -> Resistor_SMD:R_0805_2012Metric
- Y1: value 8MHz -> ATS080B-E; footprint Crystal:Crystal_HC49-U_Vertical -> Crystal:Crystal_HC49-4H_Vertical
- renumbered Q5 to Q3
Connections:
- net GNDPWR: now also R3.1
- net RCTFR+: now reaches D6.1 (+), L1.1
- net RCTFR-: now reaches D6.4 (-)
- net RCTFR-: now also R3.4
- net PFC_G: now reaches Q3.1 (G)
- new net SHUNT+: R3.2
- new net SHUNT-: R3.3
Other:
- moved on the sheet: C1, C2, D6, R2, Y1

Commit message: large amount of work
Parts:
- removed R3: 4m, symbol Device:R_Shunt
- added C14, C29: 0.1u, Capacitor_SMD:C_0805_2012Metric, symbol Device:C
- added C22: 10u film, Capacitor_THT:C_Rect_L31.5mm_W15.0mm_P27.50mm_MKS4, symbol Device:C
- added R10, R16, R17, R9: R, symbol Device:R
- added R3: 4m, Resistor_SMD:R_2512_6332Metric, symbol Device:R
- added R4: 2, Resistor_SMD:R_0805_2012Metric, symbol Device:R
- added U10: INA281A2, Package_TO_SOT_SMD:SOT-23-5, symbol Amplifier_Current:INA281A2
- added U9: MCP1407, Package_SO:SOIC-8_3.9x4.9mm_P1.27mm, symbol Driver_FET:MCP1416
- C3: value 330u -> 220u; footprint Capacitor_THT:CP_Radial_D35.0mm_P10.00mm_3pin_SnapIn -> Capacitor_THT:CP_Radial_D35.0mm_P10.00mm_SnapIn
- L1: value 470uH -> 330uH; footprint (none) -> TerminalBlock_Phoenix:TerminalBlock_Phoenix_MKDS-1,5-2_1x02_P5.00mm_Horizontal
Connections:
- net GNDPWR is gone; now on net GND: C3.2, Q3.3 (E)
- net +PWR: now also C22.1, R16.2
- net GND: now also C14.1, C22.2, C29.1, R17.1, R3.2, U10.2 (GND), U10.3 (Vin+), U9.4 (GND), U9.5 (GND)
- net PFC_G: now also R4.2
- net RCTFR+: now also R9.2
- net RCTFR-: now also R10.1, R3.1, U10.4 (Vin-)
- net PFC_PWMIN: now reaches U6.11 (PA1)
- net PFC_PWMIN: now also U9.2 (IN)
- net IL_GAINED: now reaches U6.12 (PA2)
- net IL_GAINED: now also U10.1 (OUT)
- net VAC_SENSE: now reaches U6.13 (PA3)
- net VAC_SENSE: now also R10.2, R9.1
- net VDC_SENSE: now reaches U6.14 (PA4)
- net VDC_SENSE: now also R16.1, R17.2
- net +3.3V: now reaches U6.24 (VDD)
- net +3.3V: now also U6.36 (VDD), U6.48 (VDD), U6.9 (VDDA), C29.2, U10.5 (V+)
- new net: R4.1, U9.6 (OUT), U9.7 (OUT)
- new net +12V: C14.2, U9.1 (Vdd), U9.8 (Vdd)
Other:
- note added: "PWR is to be regulated around 400V"
- note added: "RCTFR is expected max 375V"
- moved on the sheet: C1, C2, C3, D5, D6, L1, Q3, R2, U6, Y1

Commit message: tentative layout completion
Connections:
- net PFC_SWNODE: now also L1.1; no longer L1.2
- net RCTFR+: now also L1.2; no longer L1.1
Other:
- moved on the sheet: L1
Changed lines of the file:
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@@
 	(symbol
 		(lib_id "Device:L")
-		(at 184.15 44.45 90)
+		(at 184.15 44.45 270)
+		(mirror x)
 		(unit 1)
 		(exclude_from_sim no)
@@
 		(on_board yes)
 		(dnp no)
-		(fields_autoplaced yes)
 		(property "Reference" "L1"
 			(at 184.15 39.37 90)

Commit message: layout nearly complete
Parts:
- added C29, C30, C31, C32, C33: 0.1u, Capacitor_SMD:C_0805_2012Metric, symbol Device:C
- added J10: SWD, Connector_PinHeader_2.54mm:PinHeader_1x04_P2.54mm_Vertical, symbol Connector:Conn_01x04_Pin
- added R18: 10K, Resistor_SMD:R_0805_2012Metric, symbol Device:R
- renumbered C29 to C7
Connections:
- net +3.3V: now also C29.2, C30.2, C31.2, C32.2, J10.1 (Pin_1), R18.1
- net GND: now also U6.44 (BOOT0), C29.1, C30.1, C31.1, C32.1, C33.2, J10.4 (Pin_4)
- net IL_GAINED: no longer U6.12 (PA2)
- net VAC_SENSE: no longer U6.13 (PA3)
- net VDC_SENSE: no longer U6.14 (PA4)
- net SWIO: now reaches U6.34 (PA13)
- net SWIO: now also J10.2 (Pin_2)
- net SWCLK: now reaches U6.37 (PA14)
- net SWCLK: now also J10.3 (Pin_3)
- net at U6.7 (NRST): now also C33.1, R18.2
- net PFC_PWMIN: no longer names the net of U6.11 (PA1)
- net PFC_PWMIN: no longer U9.2 (IN)
- new net PFC_PWM: U9.2 (IN)
Other:
- moved on the sheet: C14, R10, R16, R17, R4, R9, U9

Commit message: tentative layout completion
Parts:
- removed C32: 0.1u, Capacitor_SMD:C_0805_2012Metric, symbol Device:C
- added C34: 10n, Capacitor_SMD:C_0805_2012Metric, symbol Device:C
- added C35: 1u, Capacitor_SMD:C_0805_2012Metric, symbol Device:C
- R10, R17: value R -> 1K HV; footprint (none) -> Resistor_SMD:R_1206_3216Metric
- R16, R9: value R -> 150K HV; footprint (none) -> Resistor_SMD:R_1206_3216Metric
Connections:
- net +3.3V: now also C34.2, C35.2
- net GND: now also C34.1, C35.1
- net IL_GAINED: now also U6.16 (PA6)
- net PFC_PWM: now also U6.14 (PA4)
- net VAC_SENSE: now also U6.15 (PA5)
- net VDC_SENSE: now also U6.13 (PA3)
- no-connect marks 0 -> 1
Other:
- moved on the sheet: C29, C30, C31

Commit message: Completed layout v1
Parts:
- added R19: 10K, Resistor_SMD:R_0805_2012Metric, symbol Device:R
Connections:
- net GND: now also R19.2
- net PFC_G: now also R19.1
Changed lines of the file:
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@@
+	)
+	(junction
+		(at 170.18 114.3)
+		(diameter 0)
+		(color 0 0 0 0)
 	)
 	(junction
@@
 	(wire
 		(pts
+			(xy 170.18 114.3) (xy 176.53 114.3)
+		)
+		(stroke
+			(width 0)
+			(type default)
+		)
+	)
+	(wire
+		(pts
 			(xy 147.32 54.61) (xy 147.32 66.04)
 		)
@@
 	(wire
 		(pts
-			(xy 166.37 114.3) (xy 176.53 114.3)
+			(xy 166.37 114.3) (xy 170.18 114.3)
 		)
 		(stroke
@@
 	(wire
 		(pts
+			(xy 170.18 114.3) (xy 170.18 116.84)
+		)
+		(stroke
+			(width 0)
+			(type default)
+		)
+	)
+	(wire
+		(pts
 			(xy 85.09 21.59) (xy 85.09 22.86)
 		)
@@
 		(pts
 			(xy 152.4 165.1) (xy 152.4 162.56)
+		)
+		(stroke
+			(width 0)
+			(type default)
+		)
+	)
+	(wire
+		(pts
+			(xy 170.18 124.46) (xy 170.18 125.73)
 		)
 		(stroke
@@
 	)
 	(symbol
+		(lib_id "Device:R")
+		(at 170.18 120.65 0)
+		(unit 1)
+		(exclude_from_sim no)
+		(in_bom yes)
+		(on_board yes)
+		(dnp no)
+		(fields_autoplaced yes)
+		(property "Reference" "R19"
+			(at 172.72 119.3799 0)
+			(effects
+				(font
+					(size 1.27 1.27)
+				)
+				(justify left)
+			)
+		)
+		(property "Value" "10K"
+			(at 172.72 121.9199 0)
+			(effects
+				(font
+					(size 1.27 1.27)
+				)
+				(justify left)
+			)
+		)
+		(property "Footprint" "Resistor_SMD:R_0805_2012Metric"
+			(at 168.402 120.65 90)
+			(effects
+				(font
+					(size 1.27 1.27)
+				)
+				(hide yes)
+			)
+		)
+		(property "Datasheet" "~"
+			(at 170.18 120.65 0)
+			(effects
+				(font
+					(size 1.27 1.27)
+				)
+				(hide yes)
+			)
+		)
+		(property "Description" "Resistor"
+			(at 170.18 120.65 0)
+			(effects
+				(font
+					(size 1.27 1.27)
+				)
+				(hide yes)
+			)
+		)
+		(pin "2"
+		)
+		(pin "1"
+		)
+		(instances
+			(project ""
+				(path "/502e07b2-2298-4bcb-9609-8c0caf105dbf/7c0adbb8-a952-4fb1-a9c1-40170fa5d3e7"
+					(reference "R19")
+					(unit 1)
+				)
+			)
+		)
+	)
+	(symbol
 		(lib_id "Device:Crystal")
 		(at 45.72 173.99 90)
@@
 					(unit 1)
 				)
+			)
+		)
+	)
+	(symbol
+		(lib_id "power:GND")
+		(at 170.18 125.73 0)
+		(unit 1)
+		(exclude_from_sim no)
+		(in_bom yes)
+		(on_board yes)
+		(dnp no)
+		(fields_autoplaced yes)
+		(property "Reference" "#PWR066"
+			(at 170.18 132.08 0)
+			(effects
+				(font
+					(size 1.27 1.27)
+				)
+				(hide yes)
+			)
+		)
+		(property "Value" "GND"
+			(at 170.18 130.81 0)
+			(effects
+				(font
+					(size 1.27 1.27)
+				)
+			)
+		)
+		(property "Footprint" ""
+			(at 170.18 125.73 0)
+			(effects
+				(font
+					(size 1.27 1.27)
+				)
+				(hide yes)
+			)
+		)
+		(property "Datasheet" ""
+			(at 170.18 125.73 0)
+			(effects
+				(font
+					(size 1.27 1.27)
+				)
+				(hide yes)
+			)
+		)
+		(property "Description" "Power symbol creates a global label with name \"GND\" , ground"
+			(at 170.18 125.73 0)
+			(effects
+				(font
+					(size 1.27 1.27)
+				)
+				(hide yes)
+			)
+		)
+		(pin "1"
+		)
+		(instances
+			(project "pfc-drsstc"
+				(path "/502e07b2-2298-4bcb-9609-8c0caf105dbf/7c0adbb8-a952-4fb1-a9c1-40170fa5d3e7"
+					(reference "#PWR066")
+					(unit 1)
+				)
