File: pfc-drsstc.kicad_pcb (KiCad board)
At the start: 2 copper layers, 109.4 x 86.4 mm, 30 parts, among them J1 12V_IN, J2 12V_IN, J3 12V_IN, J4 12V_IN, Q1 FGA60N65SMD, Q2 FGA60N65SMD, Q3 FGA60N65SMD, Q4 FGA60N65SMD, Q5 FGA60N65SMD, U1 74LS14, U2 74LS74, U3 74LS08, U4 LM311, U5 TL3116, U6 STM32F103C8Tx, U7 MCP1703Ax-330xxDB, U8 MCP1703Ax-500xxDB, Y1 8MHz

Commit message: large amount of work
Parts:
- removed the C6 at (140.8, 113.2)
- removed the Q3 at (159.2, 81.2)
- added C10: 0.1u, Capacitor_SMD:C_0805_2012Metric, F.Cu at (150.9, 115.5)
- added C11: 1uF 630V, Capacitor_THT:C_Rect_L26.5mm_W10.5mm_P22.50mm_MKS4, F.Cu at (110.6, 73.6)
- added C12: 1uF 630V, Capacitor_THT:C_Rect_L26.5mm_W10.5mm_P22.50mm_MKS4, F.Cu at (88.1, 62.6)
- added C14: 0.1u, Capacitor_SMD:C_0805_2012Metric, F.Cu at (84.4, 117.3)
- added C15: 0.1u, Capacitor_SMD:C_0805_2012Metric, F.Cu at (147.1, 136.3)
- added C16: 1n, Capacitor_SMD:C_0805_2012Metric, F.Cu at (170.0, 127.8)
- added C17: 22n, Capacitor_SMD:C_0805_2012Metric, F.Cu at (157.3, 118.0)
- added C18: 0.1u, Capacitor_SMD:C_0805_2012Metric, F.Cu at (167.2, 129.1)
- added C19: 0.1u, Capacitor_SMD:C_0805_2012Metric, F.Cu at (154.1, 135.0)
- added C20: 0.1u, Capacitor_SMD:C_0805_2012Metric, F.Cu at (170.8, 122.9)
- added C21: 1u, Capacitor_SMD:C_0805_2012Metric, F.Cu at (148.7, 80.7)
- added C22: 10u film, Capacitor_THT:C_Rect_L31.5mm_W15.0mm_P27.50mm_MKS4, F.Cu at (85.5, 102.6)
- added C23: 10u, Capacitor_SMD:C_1206_3216Metric, F.Cu at (165.0, 95.8)
- added C24: 10u, Capacitor_SMD:C_1206_3216Metric, F.Cu at (167.6, 95.8)
- added C25: 10u, Capacitor_SMD:C_1206_3216Metric, F.Cu at (161.2, 62.1)
- added C26: 10u, Capacitor_SMD:C_1206_3216Metric, F.Cu at (161.2, 82.2)
- added C27: 0.1u, Capacitor_SMD:C_0805_2012Metric, F.Cu at (154.2, 82.7)
- added C28: 0.1u, Capacitor_SMD:C_0805_2012Metric, F.Cu at (149.8, 67.3)
- added C29: 0.1u, Capacitor_SMD:C_0805_2012Metric, F.Cu at (84.6, 142.2)
- added C8: 0.1u, Capacitor_SMD:C_0805_2012Metric, F.Cu at (164.8, 112.4)
- added C9: 0.1u, Capacitor_SMD:C_0805_2012Metric, F.Cu at (150.9, 124.4)
- added D1: 1N5819, Diode_THT:D_DO-41_SOD81_P2.54mm_Vertical_AnodeUp, F.Cu at (167.2, 146.8)
- added D10: 1N5819, Diode_THT:D_DO-41_SOD81_P2.54mm_Vertical_AnodeUp, F.Cu at (149.5, 152.3)
- added D11: 1N5819, Diode_THT:D_DO-41_SOD81_P2.54mm_Vertical_AnodeUp, F.Cu at (159.3, 143.7)
- added D12: 1N5337BG, Diode_THT:D_5KPW_P7.62mm_Vertical_AnodeUp, F.Cu at (155.8, 152.3)
- added D13: 1N5337BG, Diode_THT:D_5KPW_P7.62mm_Vertical_AnodeUp, F.Cu at (152.7, 143.7)
- added D14: 1N4148, Diode_THT:D_DO-35_SOD27_P2.54mm_Vertical_AnodeUp, F.Cu at (143.5, 134.5)
- added D15: 1N5819, Diode_THT:D_DO-41_SOD81_P2.54mm_Vertical_AnodeUp, F.Cu at (80.9, 71.7)
- added D16: SD24C, Diode_SMD:D_SOD-323, F.Cu at (78.1, 75.5)
- added D17: SD24C, Diode_SMD:D_SOD-323, F.Cu at (78.4, 91.7)
- added D18: 1N4148, Diode_THT:D_DO-35_SOD27_P2.54mm_Vertical_AnodeUp, F.Cu at (148.8, 84.8)
- added D19: 1N4148, Diode_THT:D_DO-35_SOD27_P2.54mm_Vertical_AnodeUp, F.Cu at (147.9, 64.8)
- added D2: 1N5819, Diode_THT:D_DO-41_SOD81_P2.54mm_Vertical_AnodeUp, F.Cu at (170.9, 146.9)
- added D20: 1N5819, Diode_THT:D_DO-41_SOD81_P2.54mm_Vertical_AnodeUp, F.Cu at (82.6, 165.7)
- added D21: 1N5819, Diode_THT:D_DO-41_SOD81_P2.54mm_Vertical_AnodeUp, F.Cu at (82.9, 156.2)
- added D3: 1N5819, Diode_THT:D_DO-41_SOD81_P2.54mm_Vertical_AnodeUp, F.Cu at (167.2, 152.6)
- added D4: 1N5819, Diode_THT:D_DO-41_SOD81_P2.54mm_Vertical_AnodeUp, F.Cu at (170.9, 152.7)
- added D7: 1N5819, Diode_THT:D_DO-41_SOD81_P2.54mm_Vertical_AnodeUp, F.Cu at (81.0, 88.0)
- added D8: 1N4148, Diode_THT:D_DO-35_SOD27_P2.54mm_Vertical_AnodeUp, F.Cu at (150.2, 132.2)
- added D9: 1N4148, Diode_THT:D_DO-35_SOD27_P2.54mm_Vertical_AnodeUp, F.Cu at (155.0, 113.9)
- added J1: AC_IN, TerminalBlock_Phoenix:TerminalBlock_Phoenix_MKDS-1,5-2_1x02_P5.00mm_Horizontal, F.Cu at (65.5, 135.9)
- added J6: PRMY, TerminalBlock_Phoenix:TerminalBlock_Phoenix_MKDS-1,5-2_1x02_P5.00mm_Horizontal, F.Cu at (65.0, 62.5)
- added J7: PHASE_FB, TerminalBlock_Phoenix:TerminalBlock_Phoenix_MKDS-1,5-2_1x02_P5.00mm_Horizontal, F.Cu at (148.4, 162.9)
- added J8: OCP, TerminalBlock_Phoenix:TerminalBlock_Phoenix_MKDS-1,5-2_1x02_P5.00mm_Horizontal, F.Cu at (166.4, 163.4)
- added J9: IF-D95T, Package_TO_SOT_THT:TO-92_Inline_Wide, F.Cu at (171.8, 120.4)
- added L1: 330uH, TerminalBlock_Phoenix:TerminalBlock_Phoenix_MKDS-1,5-2_1x02_P5.00mm_Horizontal, F.Cu at (65.3, 119.0)
- added Q5: NMOS DPAK, Package_TO_SOT_SMD:TO-252-2, F.Cu at (158.8, 75.1)
- added Q6: PMOS DPAK, Package_TO_SOT_SMD:TO-252-2, F.Cu at (158.9, 87.2)
- added Q7: PMOS DPAK, Package_TO_SOT_SMD:TO-252-2, F.Cu at (158.8, 67.1)
- added R11: 10R 1W, Resistor_SMD:R_2512_6332Metric, F.Cu at (84.7, 90.8)
- added R12: 10R 1W, Resistor_SMD:R_2512_6332Metric, F.Cu at (84.6, 73.8)
- added R13: 10R 1W, Resistor_SMD:R_2512_6332Metric, F.Cu at (167.7, 91.1)
- added R14: 1K, Resistor_SMD:R_0805_2012Metric, F.Cu at (150.7, 87.1)
- added R15: 1K, Resistor_SMD:R_0805_2012Metric, F.Cu at (149.8, 69.5)
- added R4: 2, Resistor_SMD:R_0805_2012Metric, F.Cu at (78.7, 112.9)
- added R5: 1K, Resistor_SMD:R_0805_2012Metric, F.Cu at (147.1, 132.6)
- added R6: 1K, Resistor_SMD:R_0805_2012Metric, F.Cu at (169.9, 129.8)
- added R7: 20K, Resistor_SMD:R_0805_2012Metric, F.Cu at (157.3, 114.4)
- added R8: 1K, Resistor_SMD:R_0805_2012Metric, F.Cu at (160.5, 127.5)
- added RV1: 10K, Potentiometer_THT:Potentiometer_Bourns_3386P_Vertical, F.Cu at (160.8, 131.8)
- added U10: INA281A2, Package_TO_SOT_SMD:SOT-23-5, F.Cu at (81.7, 142.2)
- added U9: MCP1407, Package_SO:SOIC-8_3.9x4.9mm_P1.27mm, F.Cu at (84.3, 113.5)
- C3: value C_Polarized_US -> 220u; footprint Capacitor_THT:CP_Radial_D35.0mm_P10.00mm_3pin_SnapIn -> Capacitor_THT:CP_Radial_D35.0mm_P10.00mm_SnapIn; moved to B.Cu
- C4, C5: value 1u -> 10u
- C6: renamed from C7; value 1u -> 10u
- D5, D6, Q1, Q2: moved to B.Cu
- J2: value 12V_IN -> GDT_PRMY
- J3: value 12V_IN -> GDT_SCDY_A
- J4: value 12V_IN -> GDT_SCDY_B
- Q3: renamed from Q5; moved to B.Cu
- Q4: value FGA60N65SMD -> NMOS DPAK; footprint Package_TO_SOT_THT:TO-3P-3_Vertical -> Package_TO_SOT_SMD:TO-252-2
- R1: value R -> 10R 1W; footprint Resistor_SMD:R_0805_2012Metric -> Resistor_SMD:R_2512_6332Metric
- R3: value R -> 4m; footprint Resistor_SMD:R_2512_6332Metric_Pad1.40x3.35mm_HandSolder -> Resistor_SMD:R_2512_6332Metric
- U1, U2, U3: footprint Package_DIP:DIP-14_W7.62mm_Socket -> Package_SO:SOIC-14_3.9x8.7mm_P1.27mm
- U4: footprint Package_DIP:DIP-8_W7.62mm_Socket -> Package_SO:SOIC-8_3.9x4.9mm_P1.27mm
- U5: value TL3116 -> UCC27423
- Y1: value 8MHz -> ATS080B-E
- moved Q2 108.0 mm to (74.5, 70.1), turned to -90 degrees
- moved Q1 96.1 mm to (74.5, 86.2), turned to -90 degrees
- moved C4 84.0 mm to (77.7, 162.8), turned to 180 degrees
- moved U8 82.0 mm to (76.2, 164.6), turned to 180 degrees
- moved U7 80.9 mm to (76.3, 154.8), turned to 180 degrees
- moved C5 79.7 mm to (78.3, 159.7), turned to 180 degrees
- moved C6 71.2 mm to (78.1, 150.0), turned to 180 degrees
- moved J5 70.4 mm to (65.8, 157.1), turned to -90 degrees
- moved D5 69.9 mm to (74.6, 102.5), turned to -90 degrees
- moved R3 67.1 mm to (77.9, 142.3), turned to 90 degrees
- moved C2 61.7 mm to (98.3, 131.7), turned to -90 degrees
- moved C1 61.2 mm to (98.3, 128.1), turned to 90 degrees
- moved J4 54.1 mm to (169.6, 63.9), turned to 90 degrees
- moved U6 53.3 mm to (84.0, 130.0), turned to 180 degrees
- moved Y1 52.3 mm to (94.4, 127.5), turned to -90 degrees
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- renumbered J1 to J5
Connections:
- net Net-(D6--) renamed /MCU and PFC/RCTFR-
- C3 pad 2: GNDPWR -> GND
- D6 pad 1: Net-(D6-+) -> /MCU and PFC/RCTFR+
- J2 pad 1: /Power stage/DRIVER+ -> /DRIVER+
- J2 pad 2: /Power stage/DRIVER- -> /DRIVER-
- J3 pad 1: /Power stage/A- -> /A+
- J3 pad 2: /Power stage/A+ -> /A-
- J4 pad 1: /Power stage/B- -> /B+
- J4 pad 2: /Power stage/B+ -> GND
- Q1 pad 1: unconnected-(Q1-G-Pad1) -> /Power stage/PWR_G_HI
- Q1 pad 3: Net-(Q1-E) -> /A-
- Q2 pad 1: unconnected-(Q2-G-Pad1) -> /Power stage/PWR_G_LO
- Q2 pad 2: Net-(Q1-E) -> /A-
- Q2 pad 3: GNDPWR -> GND
- Q3 pad 1: unconnected-(Q5-G-Pad1) -> /MCU and PFC/PFC_G
- Q3 pad 3: GNDPWR -> GND
- Q4 pad 1: unconnected-(Q4-G-Pad1) -> /Feedback controller/UCC_OUTA
- Q4 pad 2: Net-(Q3-E) -> /Feedback controller/DRIVER+_PRECAP
- Q4 pad 3: GNDPWR -> GND
- R1 pad 1: unconnected-(R1-Pad1) -> /Feedback controller/OCP_RECTV
- R1 pad 2: unconnected-(R1-Pad2) -> GND
- R3 pad 2: GNDPWR -> GND
- U1 pad 1: unconnected-(U1-Pad1) -> Net-(U1-Pad1)
- U1 pad 10: unconnected-(U1-Pad10) -> Net-(U1-Pad10)
- U1 pad 11: unconnected-(U1-Pad11) -> /Feedback controller/INT_RAW
- U1 pad 12: unconnected-(U1-Pad12) -> Net-(U1-Pad12)
- U1 pad 13: unconnected-(U1-Pad13) -> Net-(U2B-C)
- U1 pad 2: unconnected-(U1-Pad2) -> Net-(D9-K)
- U1 pad 3: unconnected-(U1-Pad3) -> Net-(D9-A)
- U1 pad 4: unconnected-(U1-Pad4) -> Net-(U2B-~{R})
- U1 pad 5: unconnected-(U1-Pad5) -> Net-(D14-A)
- U1 pad 6: unconnected-(U1-Pad6) -> Net-(U2B-C)
- U1 pad 8: unconnected-(U1-Pad8) -> /Feedback controller/INT_SQUARED
- U1 pad 9: unconnected-(U1-Pad9) -> Net-(U1-Pad10)
- U2 pad 1: unconnected-(U2A-~{R}-Pad1) -> /Feedback controller/OCP_TRIG
- U2 pad 10: unconnected-(U2B-~{S}-Pad10) -> Net-(D9-K)
- U2 pad 11: unconnected-(U2B-C-Pad11) -> Net-(U2B-C)
- U2 pad 12: unconnected-(U2B-D-Pad12) -> GND
- U2 pad 13: unconnected-(U2B-~{R}-Pad13) -> Net-(U2B-~{R})
- U2 pad 2: unconnected-(U2A-D-Pad2) -> +5V
- U2 pad 3: unconnected-(U2A-C-Pad3) -> /Feedback controller/INT_SQUARED
- U2 pad 4: unconnected-(U2A-~{S}-Pad4) -> +5V
- U2 pad 5: unconnected-(U2A-Q-Pad5) -> /Feedback controller/nOCP
- U2 pad 9: unconnected-(U2B-Q-Pad9) -> Net-(U2B-Q)
- U3 pad 1: unconnected-(U3-Pad1) -> Net-(U2B-Q)
- U3 pad 10: unconnected-(U3-Pad10) -> /Feedback controller/nOCP
- U3 pad 12: unconnected-(U3-Pad12) -> GND
- U3 pad 13: unconnected-(U3-Pad13) -> GND
- U3 pad 2: unconnected-(U3-Pad2) -> Net-(U2B-C)
- U3 pad 3: unconnected-(U3-Pad3) -> Net-(U5-INA)
- U3 pad 4: unconnected-(U3-Pad4) -> Net-(U1-Pad12)
- U3 pad 5: unconnected-(U3-Pad5) -> Net-(U2B-Q)
- U3 pad 6: unconnected-(U3-Pad6) -> Net-(U5-INB)
- U3 pad 8: unconnected-(U3-Pad8) -> Net-(U1-Pad1)
- U3 pad 9: unconnected-(U3-Pad9) -> /Feedback controller/INT_SQUARED
- U4 pad 1: unconnected-(U4-GND-Pad1) -> GND
- U4 pad 2: unconnected-(U4-+-Pad2) -> /Feedback controller/OCP_SETPOINT
- U4 pad 3: unconnected-(U4---Pad3) -> /Feedback controller/OCP_RECTV
- U4 pad 4: unconnected-(U4-V--Pad4) -> GND
- U4 pad 5: unconnected-(U4-BAL-Pad5) -> Net-(U4-BAL)
- U4 pad 6: unconnected-(U4-STRB-Pad6) -> Net-(U4-BAL)
- U4 pad 7: unconnected-(U4-Pad7) -> /Feedback controller/OCP_TRIG
- U4 pad 8: unconnected-(U4-V+-Pad8) -> +5V
- U5 pad 1: unconnected-(U5-V+-Pad1) -> +5V
- U5 pad 2: unconnected-(U5-+-Pad2) -> Net-(U5-INA)
- U5 pad 3: unconnected-(U5---Pad3) -> GND
- U5 pad 4: unconnected-(U5-V--Pad4) -> Net-(U5-INB)
- U5 pad 5: unconnected-(U5-LATCH-Pad5) -> /Feedback controller/UCC_OUTB
- U5 pad 6: unconnected-(U5-GND-Pad6) -> +5V
- U5 pad 7: unconnected-(U5-Q-Pad7) -> /Feedback controller/UCC_OUTA
- U5 pad 8: unconnected-(U5-~{Q}-Pad8) -> +5V
- U6 pad 11: unconnected-(U6-PA1-Pad11) -> /MCU and PFC/PFC_PWMIN
- U6 pad 12: unconnected-(U6-PA2-Pad12) -> /MCU and PFC/IL_GAINED
- U6 pad 13: unconnected-(U6-PA3-Pad13) -> /MCU and PFC/VAC_SENSE
- U6 pad 14: unconnected-(U6-PA4-Pad14) -> /MCU and PFC/VDC_SENSE
- U6 pad 24: unconnected-(U6-VDD-Pad24) -> +3.3V
- U6 pad 36: unconnected-(U6-VDD-Pad36) -> +3.3V
- U6 pad 48: unconnected-(U6-VDD-Pad48) -> +3.3V
- U6 pad 9: unconnected-(U6-VDDA-Pad9) -> +3.3V
- U7 pad 1: +12V -> +5V
Other:
- board size 109.4 x 86.4 mm -> 80.8 x 111.5 mm

Commit message: tentative layout completion
Parts:
- moved J4 110.2 mm to (65.5, 100.0), turned to -90 degrees
- moved J3 104.3 mm to (65.4, 80.3), turned to -90 degrees
- moved J8 37.6 mm to (129.0, 160.5)
- moved R1 36.9 mm to (132.2, 140.4)
- moved C16 36.9 mm to (133.2, 125.2)
- moved C15 36.9 mm to (110.3, 133.6)
- moved D10 36.9 mm to (112.7, 149.7)
- moved D12 36.9 mm to (119.0, 149.7)
- moved D14 36.9 mm to (106.7, 131.8)
- moved D8 36.9 mm to (113.4, 129.5)
- moved R5 36.9 mm to (110.3, 129.9)
- moved R8 36.9 mm to (123.7, 124.8)
- moved RV1 36.9 mm to (124.0, 129.1)
- moved U1 36.9 mm to (126.0, 115.3)
- moved D13 36.9 mm to (116.0, 141.1)
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Connections:
- J1 pad 1: /MCU and PFC/MAINS_LINE -> /MCU and PFC/MAINS_NEUT
- J1 pad 2: /MCU and PFC/MAINS_NEUT -> /MCU and PFC/MAINS_LINE
- J6 pad 1: /Power stage/PWR_MIDPT -> /Power stage/LC_CAPSIDE
- J6 pad 2: /Power stage/LC_CAPSIDE -> /Power stage/PWR_MIDPT
- L1 pad 1: /MCU and PFC/RCTFR+ -> /MCU and PFC/PFC_SWNODE
- L1 pad 2: /MCU and PFC/PFC_SWNODE -> /MCU and PFC/RCTFR+
Routing:
- added copper zone on B.Cu, net GND
Other:
- board size 80.8 x 111.5 mm -> 78.3 x 108.6 mm

Commit message: layout nearly complete
Parts:
- added C29: 0.1u, Capacitor_SMD:C_0805_2012Metric, F.Cu at (138.7, 119.2)
- added C30: 0.1u, Capacitor_SMD:C_0805_2012Metric, F.Cu at (130.4, 116.0)
- added C31: 0.1u, Capacitor_SMD:C_0805_2012Metric, F.Cu at (133.6, 106.7)
- added C32: 0.1u, Capacitor_SMD:C_0805_2012Metric, F.Cu at (142.9, 111.7)
- added C33: 0.1u, Capacitor_SMD:C_0805_2012Metric, F.Cu at (143.9, 118.2)
- added J10: SWD, Connector_PinHeader_2.54mm:PinHeader_1x04_P2.54mm_Vertical, F.Cu at (126.8, 110.5)
- added R18: 10K, Resistor_SMD:R_0805_2012Metric, F.Cu at (141.8, 118.3)
- moved J5 142.0 mm to (185.3, 78.7), turned to 90 degrees
- moved D20 128.6 mm to (174.2, 71.1), turned to 180 degrees
- moved C4 128.6 mm to (178.0, 75.9), turned to -90 degrees
- moved U8 118.4 mm to (173.1, 77.6), turned to -90 degrees
- moved D21 115.7 mm to (164.5, 71.0), turned to 180 degrees
- moved C5 114.0 mm to (168.2, 75.4), turned to -90 degrees
- moved U7 104.3 mm to (163.4, 77.5), turned to -90 degrees
- moved C6 100.7 mm to (158.5, 75.6), turned to -90 degrees
- moved R8 60.3 mm to (178.5, 99.5), turned to 0 degrees
- moved J9 58.8 mm to (187.7, 91.7)
- moved C20 58.8 mm to (186.8, 94.2)
- moved R1 58.3 mm to (184.1, 114.0)
- moved J8 58.3 mm to (180.9, 134.1)
- moved R6 58.1 mm to (185.1, 101.1)
- moved C16 58.1 mm to (185.1, 99.0)
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- renumbered C29 to C7
Connections:
- J2 pad 1: /DRIVER+ -> /DRIVER-
- J2 pad 2: /DRIVER- -> /DRIVER+
- J6 pad 1: /Power stage/LC_CAPSIDE -> /Power stage/PWR_MIDPT
- J6 pad 2: /Power stage/PWR_MIDPT -> /A-
- U3 pad 1: Net-(U2B-Q) -> Net-(U1-Pad12)
- U3 pad 2: Net-(U2B-C) -> Net-(U2B-Q)
- U3 pad 3: Net-(U5-INA) -> Net-(U5-INB)
- U3 pad 4: Net-(U1-Pad12) -> Net-(U2B-Q)
- U3 pad 5: Net-(U2B-Q) -> Net-(U2B-C)
- U3 pad 6: Net-(U5-INB) -> Net-(U5-INA)
- U6 pad 34: unconnected-(U6-PA13-Pad34) -> /MCU and PFC/SWIO
- U6 pad 37: unconnected-(U6-PA14-Pad37) -> /MCU and PFC/SWCLK
- U6 pad 44: unconnected-(U6-BOOT0-Pad44) -> GND
- U6 pad 7: unconnected-(U6-NRST-Pad7) -> Net-(U6-NRST)
Routing:
- net GND: track 0.00 -> 165.5 mm, vias 0 -> 28
- net +5V: track 0.00 -> 154.9 mm, vias 0 -> 8
- net +12V: track 0.00 -> 126.7 mm, vias 0 -> 5
- net +PWR: track 0.00 -> 69.0 mm
- net /A-: track 0.00 -> 65.8 mm
- net +3.3V: track 0.00 -> 51.8 mm, vias 0 -> 2
- net Net-(U2B-C): track 0.00 -> 50.9 mm, vias 0 -> 2
- net /Feedback controller/INT_SQUARED: track 0.00 -> 40.2 mm, vias 0 -> 2
- net Net-(D14-A): track 0.00 -> 35.6 mm, vias 0 -> 1
- net /Feedback controller/OCP_TRIG: track 0.00 -> 31.7 mm, vias 0 -> 2
- net /Feedback controller/UCC_OUTB: track 0.00 -> 31.2 mm
- net /Power stage/PWR_MIDPT: track 0.00 -> 30.4 mm
- net Net-(D10-A): track 0.00 -> 26.9 mm
- net /MCU and PFC/PFC_SWNODE: track 0.00 -> 25.9 mm
- net /DRIVER-: track 0.00 -> 24.6 mm
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- added copper zone on B.Cu, net +12V
- added copper zone on F.Cu, net +12V
Other:
- board size 78.3 x 108.6 mm -> 88.3 x 100.2 mm
- board text added: "Air flows in from this direction"

Commit message: tentative layout completion
Parts:
- removed C32: 0.1u, Capacitor_SMD:C_0805_2012Metric
- added C34: 10n, Capacitor_SMD:C_0805_2012Metric, F.Cu at (139.1, 116.4)
- added C35: 1u, Capacitor_SMD:C_0805_2012Metric, F.Cu at (139.1, 118.5)
- added R10: 1K HV, Resistor_SMD:R_1206_3216Metric, F.Cu at (119.1, 118.9)
- added R16: 150K HV, Resistor_SMD:R_1206_3216Metric, F.Cu at (134.7, 94.3)
- added R17: 1K HV, Resistor_SMD:R_1206_3216Metric, F.Cu at (141.7, 94.3)
- added R9: 150K HV, Resistor_SMD:R_1206_3216Metric, F.Cu at (119.1, 113.8)
- moved J10 27.5 mm to (140.1, 134.6), turned to 90 degrees
- moved C30 20.1 mm to (143.7, 131.2), turned to 0 degrees
- moved C31 20.0 mm to (134.3, 126.6), turned to -90 degrees
- moved C1 13.3 mm to (140.3, 107.3), turned to 180 degrees
- moved U6 12.5 mm to (140.6, 124.8), turned to -90 degrees
- moved C2 12.1 mm to (143.9, 107.3), turned to 0 degrees
- moved Y1 9.20 mm to (139.7, 111.2), turned to 0 degrees
- moved C29 8.91 mm to (146.8, 122.9), turned to 90 degrees
- moved R18 5.33 mm to (146.9, 120.0), turned to 180 degrees
- moved R2 4.25 mm to (142.3, 115.7)
- moved C7 3.39 mm to (129.6, 125.0)
- moved R3 3.39 mm to (122.9, 125.2)
- moved U10 3.39 mm to (126.7, 125.1)
- moved C33 3.02 mm to (146.9, 117.9), turned to 0 degrees
Connections:
- U6 pad 11: /MCU and PFC/PFC_PWMIN -> unconnected-(U6-PA1-Pad11)
- U6 pad 12: /MCU and PFC/IL_GAINED -> unconnected-(U6-PA2-Pad12)
- U6 pad 13: /MCU and PFC/VAC_SENSE -> /MCU and PFC/VDC_SENSE
- U6 pad 14: /MCU and PFC/VDC_SENSE -> /MCU and PFC/PFC_PWM
- U6 pad 15: unconnected-(U6-PA5-Pad15) -> /MCU and PFC/VAC_SENSE
- U6 pad 16: unconnected-(U6-PA6-Pad16) -> /MCU and PFC/IL_GAINED
- U9 pad 2: /MCU and PFC/PFC_PWMIN -> /MCU and PFC/PFC_PWM
Routing:
- net +3.3V: track 51.8 -> 111.6 mm, vias 2 -> 4
- net GND: track 165.5 -> 207.8 mm, vias 28 -> 46
- net /MCU and PFC/VDC_SENSE: track 0.00 -> 33.5 mm, vias 0 -> 2
- net /MCU and PFC/PFC_PWM: track 0.00 -> 25.2 mm
- net /MCU and PFC/VAC_SENSE: track 0.00 -> 22.7 mm
- net /MCU and PFC/XIN: track 0.00 -> 14.8 mm
- net +PWR: track 69.0 -> 83.2 mm
- net /MCU and PFC/PFC_PWMIN: track 12.9 -> 0.00 mm
- net /MCU and PFC/RCTFR-: track 9.08 -> 20.2 mm
- net Net-(U6-NRST): track 0.00 -> 9.35 mm
- net Net-(C1-Pad2): track 0.00 -> 8.68 mm
- net /MCU and PFC/SWCLK: track 0.00 -> 8.34 mm
- net /MCU and PFC/SWIO: track 0.00 -> 6.39 mm
- net /MCU and PFC/XOUT: track 0.00 -> 4.73 mm
- net /MCU and PFC/RCTFR+: track 10.5 -> 15.1 mm
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- added copper zone on F.Cu, net GND

Commit message: Completed layout v1
Parts:
- added H1: MountingHole, MountingHole:MountingHole_3.2mm_M3, F.Cu at (185.4, 43.7)
- added H2: MountingHole, MountingHole:MountingHole_3.2mm_M3, F.Cu at (106.8, 134.0)
- added R19: 10K, Resistor_SMD:R_0805_2012Metric, F.Cu at (120.5, 98.1)
- C11, C12: value 1uF 630V -> 1u film
Routing:
- net /MCU and PFC/PFC_G: track 3.43 -> 5.90 mm
- net GND: track 207.8 -> 209.4 mm, vias 46 -> 47
Other:
- board text added: "3V3 IO CK GND"
- board text added: "A+"
- board text added: "A-"
- board text added: "B+"
- board text added: "B-"
- board text added: "FB"
- board text added: "GDT+"
- board text added: "GDT-"
- board text added: "INDUCTOR"
- board text added: "LINE"
- board text added: "NEUT"
- board text added: "OCP"
- board text added: "PRIMARY"
