File: pfc-drsstc.kicad_sch (KiCad schematic)
At the start: 7 parts, among them J1 12V_IN, U7 MCP1703Ax-330xxDB, U8 MCP1703Ax-500xxDB

Commit message: added progress
Parts:
- added J1: AC_IN, TerminalBlock_Phoenix:TerminalBlock_Phoenix_MKDS-1,5-2_1x02_P5.00mm_Horizontal, symbol Connector:Screw_Terminal_01x02
- renumbered J1 to J5
Connections:
- new net MAINS_LINE: J1.2 (Pin_2)
- new net MAINS_NEUT: J1.1 (Pin_1)
Changed lines of the file:
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@@
+	(wire
+		(pts
+			(xy 156.21 35.56) (xy 172.72 35.56)
+		)
+		(stroke
+			(width 0)
+			(type default)
+		)
+	)
 	(wire
 		(pts
@@
 	(wire
 		(pts
+			(xy 156.21 33.02) (xy 172.72 33.02)
+		)
+		(stroke
+			(width 0)
+			(type default)
+		)
+	)
+	(wire
+		(pts
 			(xy 180.34 93.98) (xy 193.04 93.98)
 		)
@@
 			(width 0)
 			(type default)
+		)
+	)
+	(label "MAINS_LINE"
+		(at 172.72 33.02 180)
+		(effects
+			(font
+				(size 1.27 1.27)
+			)
+			(justify right bottom)
+		)
+	)
+	(label "MAINS_NEUT"
+		(at 172.72 35.56 180)
+		(effects
+			(font
+				(size 1.27 1.27)
+			)
+			(justify right bottom)
 		)
 	)
@@
 		(dnp no)
 		(fields_autoplaced yes)
-		(property "Reference" "J1"
+		(property "Reference" "J5"
 			(at 151.13 43.18 0)
 			(effects
@@
 			(project ""
 				(path "/502e07b2-2298-4bcb-9609-8c0caf105dbf"
-					(reference "J1")
+					(reference "J5")
 					(unit 1)
 				)
@@
 					(unit 1)
 				)
+			)
+		)
+	)
+	(symbol
+		(lib_id "Connector:Screw_Terminal_01x02")
+		(at 151.13 35.56 180)
+		(unit 1)
+		(exclude_from_sim no)
+		(in_bom yes)
+		(on_board yes)
+		(dnp no)
+		(fields_autoplaced yes)
+		(property "Reference" "J1"
+			(at 151.13 26.67 0)
+			(effects
+				(font
+					(size 1.27 1.27)
+				)
+			)
+		)
+		(property "Value" "AC_IN"
+			(at 151.13 29.21 0)
+			(effects
+				(font
+					(size 1.27 1.27)
+				)
+			)
+		)
+		(property "Footprint" "TerminalBlock_Phoenix:TerminalBlock_Phoenix_MKDS-1,5-2_1x02_P5.00mm_Horizontal"
+			(at 151.13 35.56 0)
+			(effects
+				(font
+					(size 1.27 1.27)
+				)
+				(hide yes)
+			)
+		)
+		(property "Datasheet" "~"
+			(at 151.13 35.56 0)
+			(effects
+				(font
+					(size 1.27 1.27)
+				)
+				(hide yes)
+			)
+		)
+		(property "Description" "Generic screw terminal, single row, 01x02, script generated (kicad-library-utils/schlib/autogen/connector/)"
+			(at 151.13 35.56 0)
+			(effects
+				(font
+					(size 1.27 1.27)
+				)
+				(hide yes)
+			)
+		)
+		(pin "2"
+		)
+		(pin "1"
+		)
+		(instances
+			(project "pfc-drsstc"
+				(path "/502e07b2-2298-4bcb-9609-8c0caf105dbf"
+					(reference "J1")
+					(unit 1)
+				)

Commit message: large amount of work
Parts:
- removed C6: 1u, Capacitor_SMD:C_0805_2012Metric, symbol Device:C
- added D20, D21: 1N5819, Diode_THT:D_DO-41_SOD81_P2.54mm_Vertical_AnodeUp, symbol Device:D_Schottky
- added J2: GDT_PRMY, TerminalBlock_Phoenix:TerminalBlock_Phoenix_MKDS-1,5-2_1x02_P5.00mm_Horizontal, symbol Connector:Screw_Terminal_01x02
- added J3: GDT_SCDY_A, TerminalBlock_Phoenix:TerminalBlock_Phoenix_MKDS-1,5-2_1x02_P5.00mm_Horizontal, symbol Connector:Screw_Terminal_01x02
- added J4: GDT_SCDY_B, TerminalBlock_Phoenix:TerminalBlock_Phoenix_MKDS-1,5-2_1x02_P5.00mm_Horizontal, symbol Connector:Screw_Terminal_01x02
- C4, C5: value 1u -> 10u
- C6: renamed from C7; value 1u -> 10u
Connections:
- net +12V: now also D20.1 (K); no longer U7.1 (VI)
- net +3.3V: now also D21.2 (A)
- net +5V: now also U7.1 (VI), D20.2 (A), D21.1 (K)
- net MAINS_LINE renamed MCU and PFC/MAINS_NEUT
- net MAINS_NEUT renamed MCU and PFC/MAINS_LINE
- new net A+: J3.1 (Pin_1)
- new net A-: J3.2 (Pin_2)
- new net B+: J4.1 (Pin_1)
- new net B-: J4.2 (Pin_2)
- new net DRIVER+: J2.1 (Pin_1)
- new net DRIVER-: J2.2 (Pin_2)
Other:
- sheet Feedback controller ports: added DRIVER+, DRIVER-; removed none
- sheet MCU and PFC ports: added MAINS_LINE, MAINS_NEUT; removed none
- sheet Power stage ports: added GDT_A+, GDT_A-, GDT_B+, GDT_B-; removed none
- note added: "GDT wound 10:15:15"
- moved on the sheet: C6, J1, U7

Commit message: tentative layout completion
Connections:
- net MCU and PFC/MAINS_LINE: now also J1.2 (Pin_2); no longer J1.1 (Pin_1)
- net MCU and PFC/MAINS_NEUT: now also J1.1 (Pin_1); no longer J1.2 (Pin_2)
Other:
- moved on the sheet: J1
Changed lines of the file:
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@@
 	(symbol
 		(lib_id "Connector:Screw_Terminal_01x02")
-		(at 62.23 144.78 0)
-		(mirror y)
+		(at 62.23 147.32 180)
 		(unit 1)
 		(exclude_from_sim no)
@@
 		(dnp no)
 		(property "Reference" "J1"
-			(at 62.23 141.732 0)
+			(at 62.23 138.684 0)
 			(effects
 				(font
@@
 		)
 		(property "Value" "AC_IN"
-			(at 62.23 139.192 0)
+			(at 62.23 141.224 0)
 			(effects
 				(font
@@
 		)
 		(property "Footprint" "TerminalBlock_Phoenix:TerminalBlock_Phoenix_MKDS-1,5-2_1x02_P5.00mm_Horizontal"
-			(at 62.23 144.78 0)
+			(at 62.23 147.32 0)
 			(effects
 				(font
@@
 		)
 		(property "Datasheet" "~"
-			(at 62.23 144.78 0)
+			(at 62.23 147.32 0)
 			(effects
 				(font
@@
 		)
 		(property "Description" "Generic screw terminal, single row, 01x02, script generated (kicad-library-utils/schlib/autogen/connector/)"
-			(at 62.23 144.78 0)
+			(at 62.23 147.32 0)
 			(effects
 				(font

Commit message: layout nearly complete
Connections:
- net DRIVER+: now also J2.2 (Pin_2); no longer J2.1 (Pin_1)
- net DRIVER-: now also J2.1 (Pin_1); no longer J2.2 (Pin_2)
Changed lines of the file:
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@@
 	(symbol
 		(lib_id "Connector:Screw_Terminal_01x02")
-		(at 77.47 102.87 0)
+		(at 77.47 105.41 0)
+		(mirror x)
 		(unit 1)
 		(exclude_from_sim no)
@@
 		(on_board yes)
 		(dnp no)
-		(fields_autoplaced yes)
 		(property "Reference" "J2"
-			(at 80.01 102.8699 0)
+			(at 80.01 105.4101 0)
 			(effects
 				(font
@@
 		)
 		(property "Value" "GDT_PRMY"
-			(at 80.01 105.4099 0)
+			(at 80.01 102.8701 0)
 			(effects
 				(font
@@
 		)
 		(property "Footprint" "TerminalBlock_Phoenix:TerminalBlock_Phoenix_MKDS-1,5-2_1x02_P5.00mm_Horizontal"
-			(at 77.47 102.87 0)
+			(at 77.47 105.41 0)
 			(effects
 				(font
@@
 		)
 		(property "Datasheet" "~"
-			(at 77.47 102.87 0)
+			(at 77.47 105.41 0)
 			(effects
 				(font
@@
 		)
 		(property "Description" "Generic screw terminal, single row, 01x02, script generated (kicad-library-utils/schlib/autogen/connector/)"
-			(at 77.47 102.87 0)
+			(at 77.47 105.41 0)
 			(effects
 				(font

Commit message: Completed layout v1
Parts:
- added H1, H2: MountingHole, MountingHole:MountingHole_3.2mm_M3, symbol Mechanical:MountingHole
Other:
- moved on the sheet: C4, C5, C6, D20, D21, J1, J2, J3, J4, J5, U7, U8
