File: power_stage.kicad_sch (KiCad schematic)
At the start: 7 parts, among them J2 12V_IN, J3 12V_IN, J4 12V_IN, Q1 FGA60N65SMD, Q2 FGA60N65SMD, Q3 FGA60N65SMD, Q4 FGA60N65SMD

Commit message: added progress
Parts:
- removed Q3, Q4: FGA60N65SMD, Package_TO_SOT_THT:TO-3P-3_Vertical, symbol Device:Q_NIGBT_GCE
- added C11, C12: C, symbol Device:C
- J2: value 12V_IN -> GDT_PRMY
- J3: value 12V_IN -> GDT_SCDY_A
- J4: value 12V_IN -> GDT_SCDY_B
Connections:
- net +PWR: now also C11.1
- net GNDPWR: now also C12.2
- new net: C11.2, C12.1
Other:
- moved on the sheet: Q1, Q2

Commit message: large amount of work
Parts:
- removed J2: GDT_PRMY, TerminalBlock_Phoenix:TerminalBlock_Phoenix_MKDS-1,5-2_1x02_P5.00mm_Horizontal, symbol Connector:Screw_Terminal_01x02
- removed J3: GDT_SCDY_A, TerminalBlock_Phoenix:TerminalBlock_Phoenix_MKDS-1,5-2_1x02_P5.00mm_Horizontal, symbol Connector:Screw_Terminal_01x02
- removed J4: GDT_SCDY_B, TerminalBlock_Phoenix:TerminalBlock_Phoenix_MKDS-1,5-2_1x02_P5.00mm_Horizontal, symbol Connector:Screw_Terminal_01x02
- added C7: 0.1u POLYPROPYLENE, symbol Device:C
- added D15, D7: 1N5819, Diode_THT:D_DO-41_SOD81_P2.54mm_Vertical_AnodeUp, symbol Device:D_Schottky
- added D16, D17: SD24C, Diode_SMD:D_SOD-323, symbol Diode:SD24_SOD323
- added J6: PRMY, TerminalBlock_Phoenix:TerminalBlock_Phoenix_MKDS-1,5-2_1x02_P5.00mm_Horizontal, symbol Connector:Screw_Terminal_01x02
- added R11, R12: 10R 1W, Resistor_SMD:R_2512_6332Metric, symbol Device:R
- C11, C12: value C -> 1uF 630V; footprint (none) -> Capacitor_THT:C_Rect_L26.5mm_W10.5mm_P22.50mm_MKS4
Connections:
- net GNDPWR: now also D16.1 (A1)
- net PWR_MIDPT: now reaches C11.2, C12.1
- net PWR_MIDPT: now also J6.1 (Pin_1)
- net PWR_G_HI: now reaches Q1.1 (G)
- net PWR_G_HI: now also D17.2 (A2), D7.2 (A), R11.2
- net GDT_A-: now reaches Q1.3 (E), Q2.2 (C)
- net GDT_A-: now also C7.1, D17.1 (A1)
- net PWR_G_LO: now reaches Q2.1 (G)
- net PWR_G_LO: now also D15.2 (A), D16.2 (A2), R12.2
- new net GDT_A+: D7.1 (K), R11.1
- new net GDT_B+: D15.1 (K), R12.1
- new net LC_CAPSIDE: C7.2, J6.2 (Pin_2)
Other:
- note added: "Primary LC resonant ckt"
- moved on the sheet: C11, C12, Q1, Q2

Commit message: tentative layout completion
Connections:
- net LC_CAPSIDE: now also J6.1 (Pin_1); no longer J6.2 (Pin_2)
- net PWR_MIDPT: now also J6.2 (Pin_2); no longer J6.1 (Pin_1)
Other:
- moved on the sheet: J6
Changed lines of the file:
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@@
 	(symbol
 		(lib_id "Connector:Screw_Terminal_01x02")
-		(at 172.72 87.63 270)
-		(mirror x)
+		(at 170.18 87.63 90)
 		(unit 1)
 		(exclude_from_sim no)
@@
 		(dnp no)
 		(property "Reference" "J6"
-			(at 167.64 86.3599 90)
+			(at 175.26 86.3599 90)
 			(effects
 				(font
@@
 		)
 		(property "Value" "PRMY"
-			(at 167.64 88.8999 90)
+			(at 175.26 88.8999 90)
 			(effects
 				(font
@@
 		)
 		(property "Footprint" "TerminalBlock_Phoenix:TerminalBlock_Phoenix_MKDS-1,5-2_1x02_P5.00mm_Horizontal"
-			(at 172.72 87.63 0)
+			(at 170.18 87.63 0)
 			(effects
 				(font
@@
 		)
 		(property "Datasheet" "~"
-			(at 172.72 87.63 0)
+			(at 170.18 87.63 0)
 			(effects
 				(font
@@
 		)
 		(property "Description" "Generic screw terminal, single row, 01x02, script generated (kicad-library-utils/schlib/autogen/connector/)"
-			(at 172.72 87.63 0)
+			(at 170.18 87.63 0)
 			(effects
 				(font

Commit message: layout nearly complete
Parts:
- removed C7: 0.1u POLYPROPYLENE, symbol Device:C
Connections:
- net LC_CAPSIDE is gone; now on net PWR_MIDPT: J6.1 (Pin_1)
- net GDT_A-: now also J6.2 (Pin_2)
- net PWR_MIDPT: no longer J6.2 (Pin_2)
Other:
- note added: "0.1u polypropylene capacitor + primary winding in series"
- moved on the sheet: J6
Changed lines of the file:
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@@
+		)
+	)
+	(text "0.1u polypropylene capacitor + primary winding in series"
+		(exclude_from_sim no)
+		(at 161.798 102.616 0)
+		(effects
+			(font
+				(size 1.27 1.27)
+			)
 		)
 	)
@@
 	(wire
 		(pts
-			(xy 172.72 93.98) (xy 195.58 93.98)
+			(xy 162.56 93.98) (xy 195.58 93.98)
 		)
 		(stroke
@@
 	(wire
 		(pts
-			(xy 125.73 93.98) (xy 140.97 93.98)
+			(xy 125.73 93.98) (xy 160.02 93.98)
 		)
 		(stroke
@@
 	(wire
 		(pts
-			(xy 170.18 93.98) (xy 148.59 93.98)
-		)
-		(stroke
-			(width 0)
-			(type default)
-		)
-	)
-	(wire
-		(pts
 			(xy 106.68 127) (xy 125.73 127)
 		)
@@
 	(wire
 		(pts
-			(xy 172.72 93.98) (xy 172.72 92.71)
+			(xy 162.56 93.98) (xy 162.56 92.71)
 		)
 		(stroke
@@
 	(wire
 		(pts
-			(xy 170.18 92.71) (xy 170.18 93.98)
+			(xy 160.02 92.71) (xy 160.02 93.98)
 		)
 		(stroke
@@
 			)
 			(justify right bottom)
-		)
-	)
-	(label "LC_CAPSIDE"
-		(at 152.4 93.98 0)
-		(effects
-			(font
-				(size 1.27 1.27)
-			)
-			(justify left bottom)
 		)
 	)
@@
 	(symbol
 		(lib_id "Connector:Screw_Terminal_01x02")
-		(at 170.18 87.63 90)
+		(at 162.56 87.63 270)
+		(mirror x)
 		(unit 1)
 		(exclude_from_sim no)
@@
 		(dnp no)
 		(property "Reference" "J6"
-			(at 175.26 86.3599 90)
+			(at 157.48 86.3599 90)
 			(effects
 				(font
@@
 		)
 		(property "Value" "PRMY"
-			(at 175.26 88.8999 90)
+			(at 157.48 88.8999 90)
 			(effects
 				(font
@@
 		)
 		(property "Footprint" "TerminalBlock_Phoenix:TerminalBlock_Phoenix_MKDS-1,5-2_1x02_P5.00mm_Horizontal"
-			(at 170.18 87.63 0)
+			(at 162.56 87.63 0)
 			(effects
 				(font
@@
 		)
 		(property "Datasheet" "~"
-			(at 170.18 87.63 0)
+			(at 162.56 87.63 0)
 			(effects
 				(font
@@
 		)
 		(property "Description" "Generic screw terminal, single row, 01x02, script generated (kicad-library-utils/schlib/autogen/connector/)"
-			(at 170.18 87.63 0)
+			(at 162.56 87.63 0)
 			(effects
 				(font
@@
 					(unit 1)
 				)
-			)
-		)
-	)
-	(symbol
-		(lib_id "Device:C")
-		(at 144.78 93.98 90)
-		(unit 1)
-		(exclude_from_sim no)
-		(in_bom yes)
-		(on_board yes)
-		(dnp no)
-		(fields_autoplaced yes)
-		(property "Reference" "C7"
-			(at 144.78 86.36 90)
-			(effects
-				(font
-					(size 1.27 1.27)
-				)
-			)
-		)
-		(property "Value" "0.1u POLYPROPYLENE"
-			(at 144.78 88.9 90)
-			(effects
-				(font
-					(size 1.27 1.27)
-				)
-			)
-		)
-		(property "Footprint" ""
-			(at 148.59 93.0148 0)
-			(effects
-				(font
-					(size 1.27 1.27)
-				)
-				(hide yes)
-			)
-		)
-		(property "Datasheet" "~"
-			(at 144.78 93.98 0)
-			(effects
-				(font
-					(size 1.27 1.27)
-				)
-				(hide yes)
-			)
-		)
-		(property "Description" "Unpolarized capacitor"
-			(at 144.78 93.98 0)
-			(effects
-				(font
-					(size 1.27 1.27)
-				)
-				(hide yes)
-			)
-		)
-		(pin "2"
-		)
-		(pin "1"
-		)
-		(instances
-			(project ""
-				(path "/502e07b2-2298-4bcb-9609-8c0caf105dbf/7c64a56a-dc37-4d34-9dec-52255824658a"
-					(reference "C7")
-					(unit 1)
-				)

Commit message: Completed layout v1
Parts:
- C11, C12: value 1uF 630V -> 1u film
Changed lines of the file:
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@@
 			)
 		)
-		(property "Value" "1uF 630V"
+		(property "Value" "1u film"
 			(at 199.39 80.0099 0)
 			(effects
@@
 			)
 		)
-		(property "Value" "1uF 630V"
+		(property "Value" "1u film"
 			(at 199.39 114.2999 0)
 			(effects
